Commit message: Readded lidar

File: four_ws_navigation/robot_description/robots/fourth_robot.urdf.xacro (robot description, xacro)
@@ -5,7 +5,7 @@
   <xacro:include filename="$(find robot_description)/urdf/suspension/suspension.urdf.xacro"/>
   <xacro:include filename="$(find robot_description)/urdf/wheel/wheel.urdf.xacro"/>
-  <!-- <xacro:include filename="$(find robot_description)/urdf/lidar_base/lidar_base.urdf.xacro"/>
+  <xacro:include filename="$(find robot_description)/urdf/lidar_base/lidar_base.urdf.xacro"/>
   <xacro:include filename="$(find robot_description)/urdf/lidar_head/lidar_head.urdf.xacro"/>
-  <xacro:include filename="$(find robot_description)/urdf/lrf/lrf.urdf.xacro"/> -->
+  <xacro:include filename="$(find robot_description)/urdf/lrf/lrf.urdf.xacro"/>
   <!-- =============== Link & Joint =============== -->
   <!-- Base -->
@@ -15,14 +15,14 @@
   </xacro:base_v0>
   <!-- lidar_base -->
-<!--   <xacro:lidar_base_v0 parent="base_link">
+  <xacro:lidar_base_v0 parent="base_link">
 	<origin xyz="-0.022 0 0.035"/>
-  </xacro:lidar_base_v0> -->
+  </xacro:lidar_base_v0>
   <!-- lidar_head -->
-<!--   <xacro:lidar_head_v0 parent="lidar_base_link">
+  <xacro:lidar_head_v0 parent="lidar_base_link">
 	<origin xyz="0.022 0 0.0"/>
         <axis xyz="0 0 1"/>
-  </xacro:lidar_head_v0> -->
+  </xacro:lidar_head_v0>
   <!-- lrf sensor -->
-<!--   <xacro:lrf_v0 prefix = "front" parent="base_link">
+  <xacro:lrf_v0 prefix = "front" parent="base_link">
 	<origin xyz="0 0 0.083"/>
   </xacro:lrf_v0>
@@ -32,5 +32,5 @@
 	<child link="lrf_link"/>
 	<origin xyz="0 0 0.01"/>
-  </joint> -->
+  </joint>
   <!-- Suspension -->
   <!-- Front Right Sus -->
@@ -86,5 +86,5 @@
   <xacro:steering_trans_v0 prefix="rear_left"/>
   <!-- ===============  lider head Transmission =============== -->
-  <!-- <xacro:lidar_trans_v0/> -->
+  <xacro:lidar_trans_v0/>
   <!-- =============== Gazebo =============== -->
   <gazebo>
@@ -95,9 +95,9 @@
   <xacro:base_gazebo_v0/>
   <!-- lidar base -->
-  <!-- <xacro:lidar_base_gazebo_v0/> -->
+  <xacro:lidar_base_gazebo_v0/>
   <!-- lidar head -->
-  <!-- <xacro:lidar_head_gazebo_v0/> -->
+  <xacro:lidar_head_gazebo_v0/>
   <!-- lrf sensor -->
-  <!-- <xacro:lrf_gazebo_v0 prefix = "front" min_rad = "-3.14" max_rad = "3.14" min_range = "0.1" max_range = "10"/> -->
+  <xacro:lrf_gazebo_v0 prefix = "front" min_rad = "-3.14" max_rad = "3.14" min_range = "0.1" max_range = "10"/>
   <!-- Wheel -->
   <xacro:wheel_gazebo_v0 prefix="fr"/>
